File: KiCAD/hpk_5mm/sipm_tia.kicad_sch (KiCad schematic)
At the start: 10 parts, among them U1 OPA810xDBV

Commit message: flexi design
Parts:
- renumbered C1 to C5, C2 to C6, C3 to C7, C4 to C8, D1 to D2, R1 to R5, R2 to R6, R3 to R7, R4 to R8, U1 to U2
Changed lines of the file:
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@@
 		(on_board yes)
 		(dnp no)
-		(property "Reference" "R4"
+		(property "Reference" "R8"
 			(at 163.576 53.34 90)
 			(effects
@@
 		(on_board yes)
 		(dnp no)
-		(property "Reference" "R2"
+		(property "Reference" "R6"
 			(at 78.74 85.344 90)
 			(effects
@@
 		(on_board yes)
 		(dnp no)
-		(property "Reference" "U1"
+		(property "Reference" "U2"
 			(at 140.716 49.53 0)
 			(effects
@@
 		(on_board yes)
 		(dnp no)
-		(property "Reference" "#PWR05"
+		(property "Reference" "#PWR010"
 			(at 153.67 68.58 0)
 			(effects
@@
 		(dnp no)
 		(fields_autoplaced yes)
-		(property "Reference" "#PWR01"
+		(property "Reference" "#PWR06"
 			(at 69.85 71.12 0)
 			(effects
@@
 		(dnp no)
 		(fields_autoplaced yes)
-		(property "Reference" "D1"
+		(property "Reference" "D2"
 			(at 86.36 57.4674 90)
 			(effects
@@
 		(dnp no)
 		(fields_autoplaced yes)
-		(property "Reference" "#PWR02"
+		(property "Reference" "#PWR07"
 			(at 81.28 96.52 0)
 			(effects
@@
 		(dnp no)
 		(fields_autoplaced yes)
-		(property "Reference" "R1"
+		(property "Reference" "R5"
 			(at 83.82 44.4499 0)
 			(effects
@@
 		(on_board yes)
 		(dnp no)
-		(property "Reference" "C3"
+		(property "Reference" "C7"
 			(at 135.128 90.17 90)
 			(effects
@@
 		(on_board yes)
 		(dnp no)
-		(property "Reference" "C4"
+		(property "Reference" "C8"
 			(at 142.2399 72.39 90)
 			(effects
@@
 		(on_board yes)
 		(dnp no)
-		(property "Reference" "C2"
+		(property "Reference" "C6"
 			(at 128.27 41.9099 0)
 			(effects
@@
 		(on_board yes)
 		(dnp no)
-		(property "Reference" "#PWR04"
+		(property "Reference" "#PWR09"
 			(at 132.08 53.34 0)
 			(effects
@@
 		(on_board yes)
 		(dnp no)
-		(property "Reference" "R3"
+		(property "Reference" "R7"
 			(at 135.636 78.74 90)
 			(effects
@@
 		(on_board yes)
 		(dnp no)
-		(property "Reference" "#PWR03"
+		(property "Reference" "#PWR08"
 			(at 123.19 59.69 0)
 			(effects
@@
 		(dnp no)
 		(fields_autoplaced yes)
-		(property "Reference" "C1"
+		(property "Reference" "C5"
 			(at 73.66 57.1499 0)
 			(effects
