File: KiCAD/extra_4mm/hpk_5mm.kicad_pcb (KiCad board)
At the start: 2 copper layers, 20.4 x 40 mm, 30 parts, among them U1 OPA810xDBV, U2 OPA810xDBV, U3 OPA810xDBV

Commit message: flex protots
Parts:
- moved R7 4.02 mm to (153.9, 68.9)
- moved R5 4.02 mm to (156.1, 63.9)
- moved C6 4.02 mm to (156.1, 64.1)
- moved R6 4.02 mm to (155.1, 69.1)
- moved R8 4.02 mm to (152.2, 66.5)
- moved C7 4.02 mm to (156.2, 68.9)
- moved C5 4.02 mm to (154.1, 63.9)
- moved C8 4.02 mm to (153.9, 64.1)
- moved D2 4.02 mm to (155.3, 65.4)
- moved U2 4.02 mm to (155.0, 66.5)
- moved C1 3.99 mm to (136.9, 64.0)
- moved C2 3.99 mm to (139.0, 64.0)
- moved C3 3.99 mm to (139.1, 69.0)
- moved C4 3.99 mm to (136.9, 64.0)
- moved D1 3.99 mm to (138.3, 65.4)
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Routing:
- net Net-(D1-A): track 0.00 -> 2.56 mm
Other:
- board size 20.4 x 40 mm -> 24.4 x 43.4 mm
